File: KiCAD/WoodElf_02/WoodElf_02.sch (KiCad schematic (older format))
At the start: 10 parts

Commit message: updated the PCB to use a 2x2mm SMD RGB LED
hopefully this works.  i want to avoid relying solely on adafruit for their 5x2mm square RGB LED, and i needed more space to allow for the screw mounts.
Parts:
- added L1: LED_ARGB, LED_SMD:LED_Cree-PLCC4_2x2mm_CW, symbol WoodElf_01:LED_ARGB
- C1: footprint WoodElfLib:WS2811 -> WoodElf_Lib:WS2811
- DIN1, DO1, GND1, SWIN1, SWO1, VDD1: footprint WoodElfLib:BlankThrough-Hole -> WoodElf_Lib:BlankThrough-Hole
- H1: footprint WoodElfLib:Kailh_HotSwap_Socket -> WoodElf_Lib:Kailh_HotSwap_Socket
- S1: footprint WoodElfLib:SW_Cherry_MX1A_1.00u_PCB -> WoodElf_Lib:SW_Cherry_MX1A_1.00u_PCB
Connections:
- wire segments 28 -> 31
Other:
- moved on the sheet: GND1
Changed lines of the file:
@@
 F 0 "S1" H 6275 3637 60  0000 C CNN
 F 1 "Kailh_RGB_Switch" H 6275 3531 60  0000 C CNN
-F 2 "WoodElfLib:SW_Cherry_MX1A_1.00u_PCB" H 6300 3150 60  0001 C CNN
+F 2 "WoodElf_Lib:SW_Cherry_MX1A_1.00u_PCB" H 6300 3150 60  0001 C CNN
 F 3 "" H 6300 3150 60  0001 C CNN
 	1    6300 3150
@@
 F 0 "C1" H 7750 3597 60  0000 C CNN
 F 1 "WS2811" H 7750 3491 60  0000 C CNN
-F 2 "WoodElfLib:WS2811" H 7750 3400 60  0001 C CNN
+F 2 "WoodElf_Lib:WS2811" H 7750 3400 60  0001 C CNN
 F 3 "" H 7750 3400 60  0001 C CNN
 	1    7750 3250
@@
 F 0 "H1" H 6100 2725 50  0000 C CNN
 F 1 "Kailh_HotSwap_SwitchMount" H 6100 2634 50  0000 C CNN
-F 2 "WoodElfLib:Kailh_HotSwap_Socket" H 6100 2500 50  0001 C CNN
+F 2 "WoodElf_Lib:Kailh_HotSwap_Socket" H 6100 2500 50  0001 C CNN
 F 3 "" H 6100 2500 50  0001 C CNN
 	1    6100 2500
@@
 Connection ~ 5700 2600
 Wire Wire Line
-	7300 3150 6800 3150
-Wire Wire Line
-	7300 3250 6800 3250
-Wire Wire Line
-	6800 3250 6800 3300
-Wire Wire Line
-	7300 3350 6900 3350
-Wire Wire Line
-	6900 3350 6900 3450
-Wire Wire Line
-	6900 3450 6800 3450
-Wire Wire Line
-	7300 3450 7000 3450
-Wire Wire Line
-	7000 3450 7000 3650
-Wire Wire Line
-	7000 3650 5150 3650
-Wire Wire Line
-	5750 3150 5150 3150
+	6050 3600 5450 3600
 Wire Wire Line
 	8200 3350 8300 3350
@@
 F 0 "VDD1" H 9250 3200 50  0000 L CNN
 F 1 "BlankThrough-Hole" H 8950 2950 50  0000 L CNN
-F 2 "WoodElfLib:BlankThrough-Hole" H 9300 3050 50  0001 C CNN
+F 2 "WoodElf_Lib:BlankThrough-Hole" H 9300 3050 50  0001 C CNN
 F 3 "" H 9300 3050 50  0001 C CNN
 	1    9300 3050
@@
 F 0 "SWIN1" H 4800 2650 50  0000 L CNN
 F 1 "BlankThrough-Hole" H 4500 2400 50  0000 L CNN
-F 2 "WoodElfLib:BlankThrough-Hole" H 4850 2500 50  0001 C CNN
+F 2 "WoodElf_Lib:BlankThrough-Hole" H 4850 2500 50  0001 C CNN
 F 3 "" H 4850 2500 50  0001 C CNN
 	1    4850 2500
@@
 F 0 "SWO1" H 9250 2650 50  0000 L CNN
 F 1 "BlankThrough-Hole" H 8950 2400 50  0000 L CNN
-F 2 "WoodElfLib:BlankThrough-Hole" H 9300 2500 50  0001 C CNN
+F 2 "WoodElf_Lib:BlankThrough-Hole" H 9300 2500 50  0001 C CNN
 F 3 "" H 9300 2500 50  0001 C CNN
 	1    9300 2500
@@
 F 0 "DIN1" H 9200 3700 50  0000 L CNN
 F 1 "BlankThrough-Hole" H 8900 3450 50  0000 L CNN
-F 2 "WoodElfLib:BlankThrough-Hole" H 9250 3550 50  0001 C CNN
+F 2 "WoodElf_Lib:BlankThrough-Hole" H 9250 3550 50  0001 C CNN
 F 3 "" H 9250 3550 50  0001 C CNN
 	1    9250 3550
@@
 F 0 "DO1" H 9000 4100 50  0000 L CNN
 F 1 "BlankThrough-Hole" H 8700 3850 50  0000 L CNN
-F 2 "WoodElfLib:BlankThrough-Hole" H 9050 3950 50  0001 C CNN
+F 2 "WoodElf_Lib:BlankThrough-Hole" H 9050 3950 50  0001 C CNN
 F 3 "" H 9050 3950 50  0001 C CNN
 	1    9050 3950
@@
 L WoodElf_01:BlankThrough-Hole GND1
 U 1 1 5C69B783
-P 4850 3650
-F 0 "GND1" H 4800 3800 50  0000 L CNN
-F 1 "BlankThrough-Hole" H 4500 3550 50  0000 L CNN
-F 2 "WoodElfLib:BlankThrough-Hole" H 4850 3650 50  0001 C CNN
-F 3 "" H 4850 3650 50  0001 C CNN
-	1    4850 3650
-	1    0    0    -1
-$EndComp
-Text Label 5150 3150 0    50   ~ 0
+P 4900 4100
+F 0 "GND1" H 4850 4250 50  0000 L CNN
+F 1 "BlankThrough-Hole" H 4550 4000 50  0000 L CNN
+F 2 "WoodElf_Lib:BlankThrough-Hole" H 4900 4100 50  0001 C CNN
+F 3 "" H 4900 4100 50  0001 C CNN
+	1    4900 4100
+	1    0    0    -1
+$EndComp
+Text Label 5450 3600 0    50   ~ 0
 USB
 Text Label 9150 3050 2    50   ~ 0
@@
 Text Label 8600 3950 0    50   ~ 0
 DO
-Text Label 5150 3650 2    50   ~ 0
+Text Label 5200 4100 2    50   ~ 0
 GND
-Text Label 4700 3650 2    50   ~ 0
+Text Label 4750 4100 2    50   ~ 0
 GND
 Text Label 5150 2500 2    50   ~ 0
@@
 Text Label 4700 2500 2    50   ~ 0
 SWIN
+Wire Wire Line
+	5200 4100 6800 4100
+Wire Wire Line
+	6800 4100 6800 3450
+Wire Wire Line
+	6800 3450 7300 3450
+Wire Wire Line
+	6450 3800 6700 3800
+Wire Wire Line
+	6700 3800 6700 3150
+Wire Wire Line
+	6700 3150 7300 3150
+Wire Wire Line
+	6600 3600 6600 3250
+Wire Wire Line
+	6600 3250 7300 3250
+Wire Wire Line
+	6450 3600 6600 3600
+Wire Wire Line
+	6450 3400 6550 3400
+Wire Wire Line
+	6550 3400 6550 3350
+Wire Wire Line
+	6550 3350 7300 3350
+$Comp
+L WoodElf_01:LED_ARGB L1
+U 1 1 5C705190
+P 6250 3600
+F 0 "L1" H 6250 3133 50  0000 C CNN
+F 1 "LED_ARGB" H 6250 3224 50  0000 C CNN
+F 2 "LED_SMD:LED_Cree-PLCC4_2x2mm_CW" H 6250 3550 50  0001 C CNN
+F 3 "~" H 6250 3550 50  0001 C CNN
+	1    6250 3600
+	-1   0    0    1
+$EndComp
 $EndSCHEMATC
