File: KiCAD/WoodElf_01/WoodElf_01.kicad_pcb (KiCad board)
At the start: 2 copper layers, 158.8 x 139.7 mm, 92 parts, among them J1 AnalogJoystick, M1 MCP23017, M2 MCP23017, M3 MCP23017, P1 ItsyBitsyM4Express, P2 ItsyBitsyM4Express

Commit message: i cant even remember how much i changed here - a lot
Parts:
- removed C26, C27, C28, C29, C30, C31, C32, C33, C34, C35, C36, C37, C38, C39, C40, C41, C42: WS2811, WoodElfLib:WS2811
- removed M1, M2, M3: MCP23017, Housings_DIP:DIP-28_W7.62mm
- removed P2: ItsyBitsyM4Express, WoodElfLib:ItsyBitsyM4Express
- removed R1, R2, R3, R4: 10k, Resistors_SMD:R_2010_HandSoldering
- removed S26, S27, S28, S29, S30, S31, S32, S33, S34, S35, S36, S37, S38, S39, S40: Kailh_RGB_Switch, WoodElfLib:SW_Cherry_MX1A_1.00u_PCB
- added C1: WS2811, WoodElfLib:WS2811, B.Cu at (42.5, 134.0)
- added C2: WS2811, WoodElfLib:WS2811, B.Cu at (42.5, 172.1)
- added D1: D, WoodElfLib:D_2010_5025Metric_Pad1.52x2.65mm_HandSolder, B.Cu at (54.0, 153.0)
- added D10: D, WoodElfLib:D_2010_5025Metric_Pad1.52x2.65mm_HandSolder, F.Cu at (248.1, 116.3)
- added D11: D, WoodElfLib:D_2010_5025Metric_Pad1.52x2.65mm_HandSolder, F.Cu at (206.3, 132.4)
- added D12: D, WoodElfLib:D_2010_5025Metric_Pad1.52x2.65mm_HandSolder, F.Cu at (206.3, 135.7)
- added D13: D, WoodElfLib:D_2010_5025Metric_Pad1.52x2.65mm_HandSolder, F.Cu at (258.0, 82.2)
- added D14: D, WoodElfLib:D_2010_5025Metric_Pad1.52x2.65mm_HandSolder, F.Cu at (233.6, 116.2)
- added D15: D, WoodElfLib:D_2010_5025Metric_Pad1.52x2.65mm_HandSolder, F.Cu at (261.3, 114.8)
- added D16: D, WoodElfLib:D_2010_5025Metric_Pad1.52x2.65mm_HandSolder, F.Cu at (125.0, 152.9)
- added D17: D, WoodElfLib:D_2010_5025Metric_Pad1.52x2.65mm_HandSolder, F.Cu at (198.2, 139.8)
- added D18: D, WoodElfLib:D_2010_5025Metric_Pad1.52x2.65mm_HandSolder, F.Cu at (191.5, 139.8)
- added D19: D, WoodElfLib:D_2010_5025Metric_Pad1.52x2.65mm_HandSolder, F.Cu at (184.7, 139.8)
- added D2: D, WoodElfLib:D_2010_5025Metric_Pad1.52x2.65mm_HandSolder, B.Cu at (54.0, 134.0)
- added D20: D, WoodElfLib:D_2010_5025Metric_Pad1.52x2.65mm_HandSolder, F.Cu at (177.9, 139.8)
- added D21: D, WoodElfLib:D_2010_5025Metric_Pad1.52x2.65mm_HandSolder, F.Cu at (138.7, 149.9)
- added D22: D, WoodElfLib:D_2010_5025Metric_Pad1.52x2.65mm_HandSolder, F.Cu at (284.0, 68.1)
- added D23: D, WoodElfLib:D_2010_5025Metric_Pad1.52x2.65mm_HandSolder, F.Cu at (267.7, 102.1)
- added D24: D, WoodElfLib:D_2010_5025Metric_Pad1.52x2.65mm_HandSolder, F.Cu at (240.0, 131.6)
- added D25: D, WoodElfLib:D_2010_5025Metric_Pad1.52x2.65mm_HandSolder, F.Cu at (284.2, 91.4)
- added D3: D, WoodElfLib:D_2010_5025Metric_Pad1.52x2.65mm_HandSolder, B.Cu at (54.0, 172.1)
- added D4: D, WoodElfLib:D_2010_5025Metric_Pad1.52x2.65mm_HandSolder, B.Cu at (54.0, 191.1)
- added D5: D, WoodElfLib:D_2010_5025Metric_Pad1.52x2.65mm_HandSolder, F.Cu at (144.8, 164.1)
- added D6: D, WoodElfLib:D_2010_5025Metric_Pad1.52x2.65mm_HandSolder, B.Cu at (73.0, 134.0)
- added D7: D, WoodElfLib:D_2010_5025Metric_Pad1.52x2.65mm_HandSolder, B.Cu at (73.0, 153.0)
- added D8: D, WoodElfLib:D_2010_5025Metric_Pad1.52x2.65mm_HandSolder, B.Cu at (73.0, 172.1)
- added D9: D, WoodElfLib:D_2010_5025Metric_Pad1.52x2.65mm_HandSolder, B.Cu at (73.0, 191.1)
- added H1: Kailh_HotSwap_SwitchMount, WoodElfLib:Kailh_HotSwap_Socket, F.Cu at (50.8, 181.0)
- added H2: Kailh_HotSwap_SwitchMount, WoodElfLib:Kailh_HotSwap_Socket, F.Cu at (69.8, 181.0)
- C11, C12, C13, C14, C15, C16, C17, C18, C19, C20, C21, C22, C23, C24, C25: moved to F.Cu
- moved C19 193.0 mm to (271.7, 84.7), turned to 0 degrees
- moved C9 160.8 mm to (61.6, 191.1)
- moved C4 158.1 mm to (42.5, 191.1)
- moved S3 143.9 mm to (50.8, 161.9)
- moved C15 134.8 mm to (257.1, 76.9), turned to 0 degrees
- moved C8 134.4 mm to (61.6, 172.1)
- moved S7 126.9 mm to (69.8, 142.9)
- moved S4 114.1 mm to (50.8, 181.0)
- moved C22 113.7 mm to (251.9, 76.9), turned to 0 degrees
- moved C16 110.0 mm to (251.9, 84.3), turned to 0 degrees
- moved S2 109.1 mm to (50.8, 123.8)
- moved C7 108.3 mm to (61.6, 153.0)
- moved S14 106.1 mm to (220.0, 58.5)
- moved C21 105.6 mm to (195.1, 134.5), turned to 0 degrees
- moved S6 103.4 mm to (69.8, 123.8)
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Connections:
- C19 pad 4: /GND_2 -> /GND_1
- C19 pad 6: /Din_2 -> Net-(C18-Pad5)
- C19 pad 8: /USB_2 -> /USB_1
- C20 pad 4: /GND_2 -> /GND_1
- C20 pad 8: /USB_2 -> /USB_1
- C21 pad 4: /GND_2 -> /GND_1
- C21 pad 8: /USB_2 -> /USB_1
- C22 pad 4: /GND_2 -> /GND_1
- C22 pad 8: /USB_2 -> /USB_1
- C23 pad 4: /GND_2 -> /GND_1
- C23 pad 8: /USB_2 -> /USB_1
- C24 pad 4: /GND_2 -> /GND_1
- C24 pad 8: /USB_2 -> /USB_1
- C25 pad 4: /GND_2 -> /GND_1
- C25 pad 8: /USB_2 -> /USB_1
- C3 pad 5: Net-(C3-Pad5) -> Net-(C2-Pad6)
- C3 pad 6: /Din_1 -> Net-(C1-Pad5)
- C4 pad 6: Net-(C3-Pad5) -> Net-(C2-Pad5)
- J1 pad 2: /A2 -> /A0
- J1 pad 3: /A3 -> /A1
- P1 pad 10: Net-(P1-Pad10) -> /A5
- P1 pad 11: Net-(P1-Pad11) -> /SCK
- P1 pad 21: Net-(P1-Pad21) -> /GPIO#1
- P1 pad 22: /SDA_1 -> /SDA
- P1 pad 23: /SCL_1 -> /SCL
- P1 pad 5: Net-(P1-Pad5) -> /A0
- P1 pad 6: Net-(P1-Pad6) -> /A1
- P1 pad 9: Net-(P1-Pad9) -> /A4
- S1 pad 2: /GND_1 -> /GPIO#4
- S10 pad 2: /GND_1 -> /SCL
- S10 pad 3: Net-(C12-Pad1) -> Net-(C10-Pad1)
- S10 pad 5: Net-(C12-Pad2) -> Net-(C10-Pad2)
- S10 pad 6: Net-(C12-Pad3) -> Net-(C10-Pad3)
- S11 pad 2: /GND_1 -> /GPIO#3
- S11 pad 3: Net-(C13-Pad1) -> Net-(C11-Pad1)
- S11 pad 5: Net-(C13-Pad2) -> Net-(C11-Pad2)
- S11 pad 6: Net-(C13-Pad3) -> Net-(C11-Pad3)
- S12 pad 2: /GND_1 -> /GPIO#4
- S12 pad 3: Net-(C14-Pad1) -> Net-(C12-Pad1)
- S12 pad 5: Net-(C14-Pad2) -> Net-(C12-Pad2)
- S12 pad 6: Net-(C14-Pad3) -> Net-(C12-Pad3)
- S13 pad 2: /GND_1 -> /GPIO#1
- S13 pad 3: Net-(C15-Pad1) -> Net-(C13-Pad1)
- S13 pad 5: Net-(C15-Pad2) -> Net-(C13-Pad2)
- S13 pad 6: Net-(C15-Pad3) -> Net-(C13-Pad3)
- S14 pad 2: /GND_1 -> /SDA
- S14 pad 3: Net-(C16-Pad1) -> Net-(C14-Pad1)
- S14 pad 5: Net-(C16-Pad2) -> Net-(C14-Pad2)
- S14 pad 6: Net-(C16-Pad3) -> Net-(C14-Pad3)
- S15 pad 2: /GND_1 -> /SCL
- S15 pad 3: Net-(C17-Pad1) -> Net-(C15-Pad1)
- S15 pad 5: Net-(C17-Pad2) -> Net-(C15-Pad2)
- S15 pad 6: Net-(C17-Pad3) -> Net-(C15-Pad3)
- S16 pad 2: /GND_1 -> /GPIO#3
- S16 pad 3: Net-(C18-Pad1) -> Net-(C16-Pad1)
- S16 pad 5: Net-(C18-Pad2) -> Net-(C16-Pad2)
- S16 pad 6: Net-(C18-Pad3) -> Net-(C16-Pad3)
- S17 pad 2: /GND_2 -> /GPIO#4
- S17 pad 3: Net-(C19-Pad1) -> Net-(C17-Pad1)
- S17 pad 4: /USB_2 -> /USB_1
- S17 pad 5: Net-(C19-Pad2) -> Net-(C17-Pad2)
- S17 pad 6: Net-(C19-Pad3) -> Net-(C17-Pad3)
- S18 pad 2: /GND_2 -> /GPIO#1
- S18 pad 3: Net-(C20-Pad1) -> Net-(C18-Pad1)
- S18 pad 4: /USB_2 -> /USB_1
- S18 pad 5: Net-(C20-Pad2) -> Net-(C18-Pad2)
- S18 pad 6: Net-(C20-Pad3) -> Net-(C18-Pad3)
- S19 pad 2: /GND_2 -> /SDA
- S19 pad 3: Net-(C21-Pad1) -> Net-(C19-Pad1)
- S19 pad 4: /USB_2 -> /USB_1
- S19 pad 5: Net-(C21-Pad2) -> Net-(C19-Pad2)
- S19 pad 6: Net-(C21-Pad3) -> Net-(C19-Pad3)
- S2 pad 2: /GND_1 -> /GPIO#3
- S2 pad 3: Net-(C4-Pad1) -> Net-(C1-Pad1)
- S2 pad 5: Net-(C4-Pad2) -> Net-(C1-Pad2)
- S2 pad 6: Net-(C4-Pad3) -> Net-(C1-Pad3)
- S20 pad 2: /GND_2 -> /SCL
- S20 pad 3: Net-(C22-Pad1) -> Net-(C20-Pad1)
- S20 pad 4: /USB_2 -> /USB_1
- S20 pad 5: Net-(C22-Pad2) -> Net-(C20-Pad2)
- S20 pad 6: Net-(C22-Pad3) -> Net-(C20-Pad3)
- S21 pad 2: /GND_2 -> /GPIO#3
- S21 pad 3: Net-(C23-Pad1) -> Net-(C21-Pad1)
- S21 pad 4: /USB_2 -> /USB_1
- S21 pad 5: Net-(C23-Pad2) -> Net-(C21-Pad2)
- S21 pad 6: Net-(C23-Pad3) -> Net-(C21-Pad3)
- S22 pad 2: /GND_2 -> /GPIO#4
- S22 pad 3: Net-(C24-Pad1) -> Net-(C22-Pad1)
- S22 pad 4: /USB_2 -> /USB_1
- S22 pad 5: Net-(C24-Pad2) -> Net-(C22-Pad2)
- S22 pad 6: Net-(C24-Pad3) -> Net-(C22-Pad3)
- S23 pad 2: /GND_2 -> /GPIO#1
- S23 pad 3: Net-(C25-Pad1) -> Net-(C23-Pad1)
- S23 pad 4: /USB_2 -> /USB_1
- S23 pad 5: Net-(C25-Pad2) -> Net-(C23-Pad2)
- S23 pad 6: Net-(C25-Pad3) -> Net-(C23-Pad3)
- S24 pad 2: /GND_2 -> /SDA
- S24 pad 3: Net-(C26-Pad1) -> Net-(C24-Pad1)
- S24 pad 4: /USB_2 -> /USB_1
- S24 pad 5: Net-(C26-Pad2) -> Net-(C24-Pad2)
- S24 pad 6: Net-(C26-Pad3) -> Net-(C24-Pad3)
- S25 pad 2: /GND_2 -> /SCL
- S25 pad 3: Net-(C27-Pad1) -> Net-(C25-Pad1)
- S25 pad 4: /USB_2 -> /USB_1
- S25 pad 5: Net-(C27-Pad2) -> Net-(C25-Pad2)
- S25 pad 6: Net-(C27-Pad3) -> Net-(C25-Pad3)
- S3 pad 2: /GND_1 -> /GPIO#1
- S3 pad 3: Net-(C5-Pad1) -> Net-(C2-Pad1)
- S3 pad 5: Net-(C5-Pad2) -> Net-(C2-Pad2)
- S3 pad 6: Net-(C5-Pad3) -> Net-(C2-Pad3)
- S4 pad 2: /GND_1 -> /SDA
- S4 pad 3: Net-(C6-Pad1) -> Net-(C4-Pad1)
- S4 pad 5: Net-(C6-Pad2) -> Net-(C4-Pad2)
- S4 pad 6: Net-(C6-Pad3) -> Net-(C4-Pad3)
- S5 pad 2: /GND_1 -> /SCL
- S5 pad 3: Net-(C7-Pad1) -> Net-(C5-Pad1)
- S5 pad 5: Net-(C7-Pad2) -> Net-(C5-Pad2)
- S5 pad 6: Net-(C7-Pad3) -> Net-(C5-Pad3)
- S6 pad 2: /GND_1 -> /GPIO#3
- S6 pad 3: Net-(C8-Pad1) -> Net-(C6-Pad1)
- S6 pad 5: Net-(C8-Pad2) -> Net-(C6-Pad2)
- S6 pad 6: Net-(C8-Pad3) -> Net-(C6-Pad3)
- S7 pad 2: /GND_1 -> /GPIO#4
- S7 pad 3: Net-(C9-Pad1) -> Net-(C7-Pad1)
- S7 pad 5: Net-(C9-Pad2) -> Net-(C7-Pad2)
- S7 pad 6: Net-(C9-Pad3) -> Net-(C7-Pad3)
- S8 pad 2: /GND_1 -> /GPIO#1
- S8 pad 3: Net-(C10-Pad1) -> Net-(C8-Pad1)
- S8 pad 5: Net-(C10-Pad2) -> Net-(C8-Pad2)
- S8 pad 6: Net-(C10-Pad3) -> Net-(C8-Pad3)
- S9 pad 2: /GND_1 -> /SDA
- S9 pad 3: Net-(C11-Pad1) -> Net-(C9-Pad1)
- S9 pad 5: Net-(C11-Pad2) -> Net-(C9-Pad2)
- S9 pad 6: Net-(C11-Pad3) -> Net-(C9-Pad3)
Routing:
- net /USB_2: track 876.1 -> 0.00 mm, vias 38 -> 0
- net /USB_1: track 663.5 -> 24.8 mm, vias 16 -> 0
- net /GND_2: track 575.7 -> 0.00 mm, vias 25 -> 0
- net /GND_1: track 491.8 -> 0.00 mm, vias 20 -> 0
- net Net-(M2-Pad22): track 396.1 -> 0.00 mm, vias 3 -> 0
- net Net-(M2-Pad26): track 307.5 -> 0.00 mm, vias 2 -> 0
- net Net-(M2-Pad27): track 286.5 -> 0.00 mm, vias 7 -> 0
- net Net-(M3-Pad6): track 260.6 -> 0.00 mm
- net /3V3_1: track 258.1 -> 0.00 mm
- net Net-(M3-Pad2): track 244.7 -> 0.00 mm, vias 3 -> 0
- net Net-(M3-Pad3): track 231.5 -> 0.00 mm, vias 3 -> 0
- net Net-(M3-Pad7): track 208.0 -> 0.00 mm, vias 2 -> 0
- net Net-(M3-Pad4): track 172.7 -> 0.00 mm, vias 3 -> 0
- net Net-(D16-Pad2): track 167.8 -> 0.00 mm, vias 2 -> 0
- net Net-(D11-Pad2): track 154.1 -> 0.00 mm, vias 5 -> 0
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- added copper zone on B.Cu, net /GND_1
- added copper zone on F.Cu, net /USB_1
- removed copper zone on F.Cu, net /GND_1
- removed copper zone on F.Cu, net /GND_2
- removed copper zone on B.Cu, net /USB_1
- removed copper zone on B.Cu, net /USB_2
Other:
- board outline removed

Commit message: fleshing out some more of the pcb
Parts:
- added C26: WS2811, WoodElfLib:WS2811, B.Cu at (137.8, 125.1)
- added C27: WS2811, WoodElfLib:WS2811, B.Cu at (137.8, 148.6)
- added C28: WS2811, WoodElfLib:WS2811, B.Cu at (137.8, 167.6)
- added C29: WS2811, WoodElfLib:WS2811, B.Cu at (137.8, 186.7)
- added C30: WS2811, WoodElfLib:WS2811, B.Cu at (137.8, 205.7)
- added C31: WS2811, WoodElfLib:WS2811, F.Cu at (88.0, 24.6)
- added C32: WS2811, WoodElfLib:WS2811, F.Cu at (273.1, 192.4)
- added C33: WS2811, WoodElfLib:WS2811, F.Cu at (71.6, 36.4)
- added C34: WS2811, WoodElfLib:WS2811, F.Cu at (82.8, 24.6)
- added C35: WS2811, WoodElfLib:WS2811, F.Cu at (281.6, 198.1)
- added C36: WS2811, WoodElfLib:WS2811, F.Cu at (259.7, 205.1)
- added C37: WS2811, WoodElfLib:WS2811, F.Cu at (76.8, 36.4)
- added C38: WS2811, WoodElfLib:WS2811, F.Cu at (301.0, 191.1)
- added C39: WS2811, WoodElfLib:WS2811, F.Cu at (267.6, 207.2)
- added C40: WS2811, WoodElfLib:WS2811, F.Cu at (99.2, 13.7)
- added D26: D, Diode_SMD:D_2010_5025Metric_Pad1.52x2.65mm_HandSolder, B.Cu at (149.2, 125.1)
- added D27: D, Diode_SMD:D_2010_5025Metric_Pad1.52x2.65mm_HandSolder, B.Cu at (149.2, 148.6)
- added D28: D, Diode_SMD:D_2010_5025Metric_Pad1.52x2.65mm_HandSolder, B.Cu at (149.2, 167.6)
- added D29: D, Diode_SMD:D_2010_5025Metric_Pad1.52x2.65mm_HandSolder, B.Cu at (149.2, 186.7)
- added D30: D, Diode_SMD:D_2010_5025Metric_Pad1.52x2.65mm_HandSolder, B.Cu at (149.2, 205.7)
- added D31: D, Diode_SMD:D_2010_5025Metric_Pad1.52x2.65mm_HandSolder, F.Cu at (47.6, 37.2)
- added D32: D, Diode_SMD:D_2010_5025Metric_Pad1.52x2.65mm_HandSolder, F.Cu at (83.7, 30.0)
- added D33: D, Diode_SMD:D_2010_5025Metric_Pad1.52x2.65mm_HandSolder, F.Cu at (-6.74, 37.2)
- added D34: D, Diode_SMD:D_2010_5025Metric_Pad1.52x2.65mm_HandSolder, F.Cu at (0.05, 37.2)
- added D35: D, Diode_SMD:D_2010_5025Metric_Pad1.52x2.65mm_HandSolder, F.Cu at (6.84, 37.2)
- added D36: D, Diode_SMD:D_2010_5025Metric_Pad1.52x2.65mm_HandSolder, F.Cu at (13.6, 37.2)
- added D37: D, Diode_SMD:D_2010_5025Metric_Pad1.52x2.65mm_HandSolder, F.Cu at (20.4, 37.2)
- added D38: D, Diode_SMD:D_2010_5025Metric_Pad1.52x2.65mm_HandSolder, F.Cu at (27.2, 37.2)
- added D39: D, Diode_SMD:D_2010_5025Metric_Pad1.52x2.65mm_HandSolder, F.Cu at (34.0, 37.2)
- added D40: D, Diode_SMD:D_2010_5025Metric_Pad1.52x2.65mm_HandSolder, F.Cu at (40.8, 37.2)
- added H10: Kailh_HotSwap_SwitchMount, WoodElfLib:Kailh_HotSwap_Socket, F.Cu at (69.8, 200.0)
- added H11: Kailh_HotSwap_SwitchMount, WoodElfLib:Kailh_HotSwap_Socket, F.Cu at (88.9, 114.9)
- added H12: Kailh_HotSwap_SwitchMount, WoodElfLib:Kailh_HotSwap_Socket, F.Cu at (88.9, 138.4)
- added H13: Kailh_HotSwap_SwitchMount, WoodElfLib:Kailh_HotSwap_Socket, F.Cu at (88.9, 157.5)
- added H14: Kailh_HotSwap_SwitchMount, WoodElfLib:Kailh_HotSwap_Socket, F.Cu at (88.9, 176.5)
- added H15: Kailh_HotSwap_SwitchMount, WoodElfLib:Kailh_HotSwap_Socket, F.Cu at (88.9, 195.6)
- added H16: Kailh_HotSwap_SwitchMount, WoodElfLib:Kailh_HotSwap_Socket, F.Cu at (108.0, 119.4)
- added H17: Kailh_HotSwap_SwitchMount, WoodElfLib:Kailh_HotSwap_Socket, F.Cu at (108.0, 142.9)
- added H18: Kailh_HotSwap_SwitchMount, WoodElfLib:Kailh_HotSwap_Socket, F.Cu at (108.0, 161.9)
- added H19: Kailh_HotSwap_SwitchMount, WoodElfLib:Kailh_HotSwap_Socket, F.Cu at (108.0, 181.0)
- added H20: Kailh_HotSwap_SwitchMount, WoodElfLib:Kailh_HotSwap_Socket, F.Cu at (108.0, 200.0)
- added H21: Kailh_HotSwap_SwitchMount, WoodElfLib:Kailh_HotSwap_Socket, F.Cu at (127.0, 114.9)
- added H22: Kailh_HotSwap_SwitchMount, WoodElfLib:Kailh_HotSwap_Socket, F.Cu at (127.0, 138.4)
- added H23: Kailh_HotSwap_SwitchMount, WoodElfLib:Kailh_HotSwap_Socket, F.Cu at (127.0, 157.5)
- added H24: Kailh_HotSwap_SwitchMount, WoodElfLib:Kailh_HotSwap_Socket, F.Cu at (127.0, 176.5)
- added H25: Kailh_HotSwap_SwitchMount, WoodElfLib:Kailh_HotSwap_Socket, F.Cu at (127.0, 195.6)
- added H26: Kailh_HotSwap_SwitchMount, WoodElfLib:Kailh_HotSwap_Socket, F.Cu at (146.1, 114.9)
- added H27: Kailh_HotSwap_SwitchMount, WoodElfLib:Kailh_HotSwap_Socket, F.Cu at (146.1, 138.4)
- added H28: Kailh_HotSwap_SwitchMount, WoodElfLib:Kailh_HotSwap_Socket, F.Cu at (146.1, 157.5)
- added H29: Kailh_HotSwap_SwitchMount, WoodElfLib:Kailh_HotSwap_Socket, F.Cu at (146.1, 176.5)
- added H3: Kailh_HotSwap_SwitchMount, WoodElfLib:Kailh_HotSwap_Socket, F.Cu at (50.8, 161.9)
- added H30: Kailh_HotSwap_SwitchMount, WoodElfLib:Kailh_HotSwap_Socket, F.Cu at (146.1, 195.6)
- added H31: Kailh_HotSwap_SwitchMount, WoodElfLib:Kailh_HotSwap_Socket, F.Cu at (58.8, 31.5)
- added H32: Kailh_HotSwap_SwitchMount, WoodElfLib:Kailh_HotSwap_Socket, F.Cu at (75.2, 17.8)
- added H33: Kailh_HotSwap_SwitchMount, WoodElfLib:Kailh_HotSwap_Socket, F.Cu at (94.4, -1.44)
- added H34: Kailh_HotSwap_SwitchMount, WoodElfLib:Kailh_HotSwap_Socket, F.Cu at (305.3, 91.8)
- added H35: Kailh_HotSwap_SwitchMount, WoodElfLib:Kailh_HotSwap_Socket, F.Cu at (75.2, 6.80)
- added H36: Kailh_HotSwap_SwitchMount, WoodElfLib:Kailh_HotSwap_Socket, F.Cu at (324.5, 83.6)
- added H37: Kailh_HotSwap_SwitchMount, WoodElfLib:Kailh_HotSwap_Socket, F.Cu at (324.5, 78.1)
- added H38: Kailh_HotSwap_SwitchMount, WoodElfLib:Kailh_HotSwap_Socket, F.Cu at (276.8, 166.6)
- added H39: Kailh_HotSwap_SwitchMount, WoodElfLib:Kailh_HotSwap_Socket, F.Cu at (324.5, 72.6)
- added H4: Kailh_HotSwap_SwitchMount, WoodElfLib:Kailh_HotSwap_Socket, F.Cu at (50.8, 181.0)
- added H40: Kailh_HotSwap_SwitchMount, WoodElfLib:Kailh_HotSwap_Socket, F.Cu at (58.8, -1.40)
- added H5: Kailh_HotSwap_SwitchMount, WoodElfLib:Kailh_HotSwap_Socket, F.Cu at (50.8, 200.0)
- added H6: Kailh_HotSwap_SwitchMount, WoodElfLib:Kailh_HotSwap_Socket, F.Cu at (69.8, 119.4)
- added H7: Kailh_HotSwap_SwitchMount, WoodElfLib:Kailh_HotSwap_Socket, F.Cu at (69.8, 142.9)
- added H8: Kailh_HotSwap_SwitchMount, WoodElfLib:Kailh_HotSwap_Socket, F.Cu at (69.8, 161.9)
- added H9: Kailh_HotSwap_SwitchMount, WoodElfLib:Kailh_HotSwap_Socket, F.Cu at (69.8, 181.0)
- added S26: Kailh_RGB_Switch, WoodElfLib:SW_Cherry_MX1A_1.00u_PCB, F.Cu at (146.1, 114.9)
- added S27: Kailh_RGB_Switch, WoodElfLib:SW_Cherry_MX1A_1.00u_PCB, F.Cu at (146.1, 138.4)
- added S28: Kailh_RGB_Switch, WoodElfLib:SW_Cherry_MX1A_1.00u_PCB, F.Cu at (146.1, 157.5)
- added S29: Kailh_RGB_Switch, WoodElfLib:SW_Cherry_MX1A_1.00u_PCB, F.Cu at (146.1, 176.5)
- added S30: Kailh_RGB_Switch, WoodElfLib:SW_Cherry_MX1A_1.00u_PCB, F.Cu at (146.1, 195.6)
- added S31: Kailh_RGB_Switch, WoodElfLib:SW_Cherry_MX1A_1.00u_PCB, F.Cu at (165.1, 119.4)
- added S32: Kailh_RGB_Switch, WoodElfLib:SW_Cherry_MX1A_1.00u_PCB, F.Cu at (229.3, 94.8)
- added S33: Kailh_RGB_Switch, WoodElfLib:SW_Cherry_MX1A_1.00u_PCB, F.Cu at (248.5, 75.6)
- added S34: Kailh_RGB_Switch, WoodElfLib:SW_Cherry_MX1A_1.00u_PCB, F.Cu at (1.98, 1.65)
- added S35: Kailh_RGB_Switch, WoodElfLib:SW_Cherry_MX1A_1.00u_PCB, F.Cu at (248.5, 94.8)
- added S36: Kailh_RGB_Switch, WoodElfLib:SW_Cherry_MX1A_1.00u_PCB, F.Cu at (267.7, 75.6)
- added S37: Kailh_RGB_Switch, WoodElfLib:SW_Cherry_MX1A_1.00u_PCB, F.Cu at (1.98, 20.8)
- added S38: Kailh_RGB_Switch, WoodElfLib:SW_Cherry_MX1A_1.00u_PCB, F.Cu at (21.2, 1.65)
- added S39: Kailh_RGB_Switch, WoodElfLib:SW_Cherry_MX1A_1.00u_PCB, F.Cu at (267.7, 94.8)
- added S40: Kailh_RGB_Switch, WoodElfLib:SW_Cherry_MX1A_1.00u_PCB, F.Cu at (286.9, 75.6)
- C11, C12, C13, C14, C15, C16, C17, C18, C19, C20, C21, C22, C23, C24, C25, D10, D11, D12, D13, D14, D15, D16, D17, D18, D19, D20, D21, D22, D23, D24, D25, D5, P1: moved to B.Cu
- moved S10 220.7 mm to (69.8, 200.0)
- moved C15 218.5 mm to (80.6, 205.7), turned to 180 degrees
- moved S5 211.3 mm to (50.8, 200.0)
- moved C19 202.3 mm to (99.7, 191.1), turned to 180 degrees
- moved D10 198.7 mm to (73.0, 210.2), turned to 90 degrees
- moved C10 197.9 mm to (61.6, 210.2), turned to 180 degrees
- moved C24 197.4 mm to (118.7, 186.7), turned to 180 degrees
- moved D15 192.1 mm to (92.1, 205.7), turned to 90 degrees
- moved D25 191.8 mm to (130.2, 205.7), turned to 90 degrees
- moved D13 186.6 mm to (92.1, 167.6), turned to 90 degrees
- moved S14 176.4 mm to (88.9, 176.5)
- moved D22 173.6 mm to (130.2, 148.6), turned to 90 degrees
- moved C16 158.8 mm to (99.7, 129.5), turned to 180 degrees
- moved D14 158.1 mm to (92.1, 186.7), turned to 90 degrees
- moved J1 154.0 mm to (220.3, 14.5)
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Connections:
- H1 pad 1: Net-(D4-Pad2) -> Net-(D2-Pad2)
- H1 pad 2: /SDA -> /GPIO#3
- H2 pad 1: Net-(D9-Pad2) -> Net-(D1-Pad2)
- H2 pad 2: /SDA -> /GPIO#4
- P1 pad 12: Net-(P1-Pad12) -> /MO
- P1 pad 13: Net-(P1-Pad13) -> /MI
- P1 pad 14: Net-(P1-Pad14) -> /GPIO#2
- S1 pad 1: Net-(D1-Pad2) -> Net-(D2-Pad2)
- S1 pad 2: /GPIO#4 -> /GPIO#3
- S1 pad 3: Net-(C3-Pad1) -> Net-(C1-Pad1)
- S1 pad 5: Net-(C3-Pad2) -> Net-(C1-Pad2)
- S1 pad 6: Net-(C3-Pad3) -> Net-(C1-Pad3)
- S2 pad 1: Net-(D2-Pad2) -> Net-(D1-Pad2)
- S2 pad 2: /GPIO#3 -> /GPIO#4
- S2 pad 3: Net-(C1-Pad1) -> Net-(C3-Pad1)
- S2 pad 5: Net-(C1-Pad2) -> Net-(C3-Pad2)
- S2 pad 6: Net-(C1-Pad3) -> Net-(C3-Pad3)
Routing:
- net /USB_1: track 24.8 -> 190.4 mm
- net /A4: track 0.00 -> 129.7 mm
- net Net-(C20-Pad5): track 0.00 -> 123.8 mm
- net Net-(C10-Pad5): track 0.00 -> 123.5 mm
- net Net-(C25-Pad5): track 0.00 -> 119.8 mm
- net Net-(C5-Pad5): track 0.00 -> 117.5 mm
- net Net-(C15-Pad5): track 0.00 -> 115.2 mm
- net /A5: track 0.00 -> 88.1 mm
- net /MO: track 0.00 -> 87.9 mm
- net /SCK: track 0.00 -> 87.9 mm
- net /SCL: track 0.00 -> 87.8 mm
- net Net-(C11-Pad5): track 0.00 -> 66.7 mm
- net /GPIO#3: track 55.6 -> 101.5 mm
- net /GPIO#4: track 77.3 -> 105.7 mm
- net Net-(C1-Pad5): track 0.00 -> 25.2 mm
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Other:
- net class Default: clearance 0.2 -> 0.1524; trace_width 0.25 -> 0.1524
- rule trace_clearance: 0.2 -> 0.1524
- rule trace_min: 0.25 -> 0.1524

Commit message: more work on the PCB design.
It's probably done at this point
Parts:
- C31, C32, C33, C34, C35, C36, C37, C38, C39, C40, D31, D32, D33, D34, D35, D36, D37, D38, D39, D40: moved to B.Cu
- moved S34 183.9 mm to (151.1, 109.2)
- moved D35 178.9 mm to (154.3, 138.4), turned to 90 degrees
- moved C36 176.8 mm to (161.9, 57.8), turned to 180 degrees
- moved S37 175.6 mm to (170.2, 71.1)
- moved D34 174.8 mm to (154.3, 119.4), turned to 90 degrees
- moved S38 173.3 mm to (170.2, 90.2)
- moved D33 173.0 mm to (154.3, 100.3), turned to 90 degrees
- moved C32 171.2 mm to (142.9, 81.3), turned to 180 degrees
- moved H40 170.9 mm to (170.2, 128.3)
- moved D40 166.8 mm to (173.4, 138.4), turned to 90 degrees
- moved C38 166.1 mm to (161.9, 100.3), turned to 180 degrees
- moved D39 161.8 mm to (173.4, 119.4), turned to 90 degrees
- moved D36 161.0 mm to (173.4, 57.8), turned to 90 degrees
- moved D38 159.2 mm to (173.4, 100.3), turned to 90 degrees
- moved D37 159.2 mm to (173.4, 81.3), turned to 90 degrees
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Routing:
- net /GPIO#2: track 0.00 -> 222.8 mm
- net /MI: track 0.00 -> 207.0 mm
- net /SCL: track 87.8 -> 280.6 mm
- net /SDA: track 101.5 -> 262.8 mm
- net /GPIO#1: track 102.4 -> 246.9 mm
- net /GPIO#4: track 105.7 -> 234.6 mm
- net Net-(C35-Pad5): track 0.00 -> 120.5 mm
- net Net-(C30-Pad5): track 0.00 -> 116.4 mm
- net /MO: track 87.9 -> 189.1 mm
- net /SCK: track 87.9 -> 170.6 mm
- net /GPIO#3: track 101.5 -> 181.8 mm
- net /A5: track 88.1 -> 155.5 mm
- net /USB_1: track 190.4 -> 245.3 mm
- net /A2: track 87.8 -> 129.5 mm
- net Net-(C11-Pad5): track 66.7 -> 25.2 mm
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Other:
- board outline added: 154.3 x 119.4 mm
- board text added: "Wood Elf Prototype 01 Grace 2019"

Commit message: Started on a full-size PCB
Parts:
- removed C1, C10, C11, C12, C13, C14, C15, C16, C17, C18, C19, C2, C20, C21, C22, C23, C24, C25, C26, C27, C28, C29, C3, C30, C31, C32, C33, C34, C35, C36, C37, C38, C39, C4, C40, C5, C6, C7, C8, C9: WS2811, WoodElfLib:WS2811
- removed D26, D27, D28, D29, D30, D31, D32, D33, D34, D35, D36, D37, D38, D39, D40: D, Diode_SMD:D_2010_5025Metric_Pad1.52x2.65mm_HandSolder
- removed H26, H27, H28, H29, H30, H31, H32, H33, H34, H35, H36, H37, H38, H39, H40: Kailh_HotSwap_SwitchMount, WoodElfLib:Kailh_HotSwap_Socket
- removed J1: AnalogJoystick, WoodElfLib:Joystick
- removed Logo_2 (x2): Wood Elf, WoodElfLib:WoodElfLogo
- removed P1: ItsyBitsyM4Express, WoodElfLib:ItsyBitsyM4Express
- removed S26, S27, S28, S29, S30, S31, S32, S33, S34, S35, S36, S37, S38, S39, S40: Kailh_RGB_Switch, WoodElfLib:SW_Cherry_MX1A_1.00u_PCB
- added G***: Tiefling_Logo, WoodElf_Lib:Tiefling_Logo, F.Cu at (174.6, 151.2)
- added L1: SK6812MINI, WoodElf_Lib:LED_SK6812MINI_PLCC4_3.5x3.5mm_P1.75mm, F.Cu at (109.5, 72.8)
- added L10: SK6812MINI, WoodElf_Lib:LED_SK6812MINI_PLCC4_3.5x3.5mm_P1.75mm, F.Cu at (109.5, 91.8)
- added L11: SK6812MINI, WoodElf_Lib:LED_SK6812MINI_PLCC4_3.5x3.5mm_P1.75mm, F.Cu at (109.5, 110.8)
- added L12: SK6812MINI, WoodElf_Lib:LED_SK6812MINI_PLCC4_3.5x3.5mm_P1.75mm, F.Cu at (128.5, 106.1)
- added L13: SK6812MINI, WoodElf_Lib:LED_SK6812MINI_PLCC4_3.5x3.5mm_P1.75mm, F.Cu at (147.5, 110.8)
- added L14: SK6812MINI, WoodElf_Lib:LED_SK6812MINI_PLCC4_3.5x3.5mm_P1.75mm, F.Cu at (166.5, 106.1)
- added L15: SK6812MINI, WoodElf_Lib:LED_SK6812MINI_PLCC4_3.5x3.5mm_P1.75mm, F.Cu at (185.5, 106.1)
- added L16: SK6812MINI, WoodElf_Lib:LED_SK6812MINI_PLCC4_3.5x3.5mm_P1.75mm, F.Cu at (185.5, 125.1)
- added L17: SK6812MINI, WoodElf_Lib:LED_SK6812MINI_PLCC4_3.5x3.5mm_P1.75mm, F.Cu at (166.5, 125.1)
- added L18: SK6812MINI, WoodElf_Lib:LED_SK6812MINI_PLCC4_3.5x3.5mm_P1.75mm, F.Cu at (147.5, 129.8)
- added L19: SK6812MINI, WoodElf_Lib:LED_SK6812MINI_PLCC4_3.5x3.5mm_P1.75mm, F.Cu at (128.5, 125.1)
- added L2: SK6812MINI, WoodElf_Lib:LED_SK6812MINI_PLCC4_3.5x3.5mm_P1.75mm, F.Cu at (128.5, 68.1)
- added L20: SK6812MINI, WoodElf_Lib:LED_SK6812MINI_PLCC4_3.5x3.5mm_P1.75mm, F.Cu at (109.5, 129.8)
- added L21: SK6812MINI, WoodElf_Lib:LED_SK6812MINI_PLCC4_3.5x3.5mm_P1.75mm, F.Cu at (109.5, 148.8)
- added L22: SK6812MINI, WoodElf_Lib:LED_SK6812MINI_PLCC4_3.5x3.5mm_P1.75mm, F.Cu at (128.5, 144.1)
- added L23: SK6812MINI, WoodElf_Lib:LED_SK6812MINI_PLCC4_3.5x3.5mm_P1.75mm, F.Cu at (147.5, 148.8)
- added L24: SK6812MINI, WoodElf_Lib:LED_SK6812MINI_PLCC4_3.5x3.5mm_P1.75mm, F.Cu at (166.5, 144.1)
- added L25: SK6812MINI, WoodElf_Lib:LED_SK6812MINI_PLCC4_3.5x3.5mm_P1.75mm, F.Cu at (185.5, 144.1)
- added L3: SK6812MINI, WoodElf_Lib:LED_SK6812MINI_PLCC4_3.5x3.5mm_P1.75mm, F.Cu at (147.5, 72.8)
- added L4: SK6812MINI, WoodElf_Lib:LED_SK6812MINI_PLCC4_3.5x3.5mm_P1.75mm, F.Cu at (166.5, 68.1)
- added L5: SK6812MINI, WoodElf_Lib:LED_SK6812MINI_PLCC4_3.5x3.5mm_P1.75mm, F.Cu at (185.5, 68.1)
- added L6: SK6812MINI, WoodElf_Lib:LED_SK6812MINI_PLCC4_3.5x3.5mm_P1.75mm, F.Cu at (185.5, 87.1)
- added L7: SK6812MINI, WoodElf_Lib:LED_SK6812MINI_PLCC4_3.5x3.5mm_P1.75mm, F.Cu at (166.5, 87.1)
- added L8: SK6812MINI, WoodElf_Lib:LED_SK6812MINI_PLCC4_3.5x3.5mm_P1.75mm, F.Cu at (147.5, 91.8)
- added L9: SK6812MINI, WoodElf_Lib:LED_SK6812MINI_PLCC4_3.5x3.5mm_P1.75mm, F.Cu at (128.5, 87.1)
- added T1: BlankThrough-Hole, WoodElf_Lib:BlankThrough-Hole, F.Cu at (141.0, 58.0)
- added T10: BlankThrough-Hole, WoodElf_Lib:BlankThrough-Hole, F.Cu at (141.0, 54.9)
- added T11: BlankThrough-Hole, WoodElf_Lib:BlankThrough-Hole, F.Cu at (153.0, 58.0)
- added T12: BlankThrough-Hole, WoodElf_Lib:BlankThrough-Hole, F.Cu at (151.0, 54.9)
- added T13: BlankThrough-Hole, WoodElf_Lib:BlankThrough-Hole, F.Cu at (151.0, 58.0)
- added T2: BlankThrough-Hole, WoodElf_Lib:BlankThrough-Hole, F.Cu at (143.0, 58.0)
- added T3: BlankThrough-Hole, WoodElf_Lib:BlankThrough-Hole, F.Cu at (145.0, 58.0)
- added T4: BlankThrough-Hole, WoodElf_Lib:BlankThrough-Hole, F.Cu at (147.0, 58.0)
- added T5: BlankThrough-Hole, WoodElf_Lib:BlankThrough-Hole, F.Cu at (149.0, 58.0)
- added T6: BlankThrough-Hole, WoodElf_Lib:BlankThrough-Hole, F.Cu at (149.0, 55.0)
- added T7: BlankThrough-Hole, WoodElf_Lib:BlankThrough-Hole, F.Cu at (147.0, 55.0)
- added T8: BlankThrough-Hole, WoodElf_Lib:BlankThrough-Hole, F.Cu at (145.0, 55.0)
- added T9: BlankThrough-Hole, WoodElf_Lib:BlankThrough-Hole, F.Cu at (143.0, 55.0)
- D1, D10, D11, D12, D13, D14, D15, D16, D17, D18, D19, D2, D20, D21, D22, D23, D24, D25, D3, D4, D5, D6, D7, D8, D9: value D -> DIODE; footprint WoodElfLib:D_2010_5025Metric_Pad1.52x2.65mm_HandSolder -> Diode_SMD:D_2010_5025Metric_Pad1.52x2.65mm_HandSolder
- H1, H10, H11, H12, H13, H14, H15, H16, H17, H18, H19, H2, H20, H21, H22, H23, H24, H25, H3, H4, H5, H6, H7, H8, H9: footprint WoodElfLib:Kailh_HotSwap_Socket -> WoodElf_Lib:Kailh_HotSwap_Socket
- S1, S10, S11, S12, S13, S14, S15, S16, S17, S18, S19, S2, S20, S21, S22, S23, S24, S25, S3, S4, S5, S6, S7, S8, S9: footprint WoodElfLib:SW_Cherry_MX1A_1.00u_PCB -> WoodElf_Lib:SW_Cherry_MX1A_1.00u_PCB
- moved D5 166.5 mm to (190.8, 67.8), turned to 270 degrees
- moved H5 166.3 mm to (187.5, 58.0)
- moved S5 166.3 mm to (187.5, 58.0)
- moved D4 141.6 mm to (171.8, 67.8), turned to 270 degrees
- moved H4 141.3 mm to (168.5, 58.0)
- moved S4 141.3 mm to (168.5, 58.0)
- moved D6 134.9 mm to (190.8, 86.8), turned to 270 degrees
- moved H6 134.9 mm to (187.5, 77.0)
- moved S6 134.9 mm to (187.5, 77.0)
- moved D15 116.2 mm to (190.8, 105.8), turned to 270 degrees
- moved D3 116.2 mm to (152.8, 72.6), turned to 270 degrees
- moved H15 116.0 mm to (187.5, 96.0)
- moved S15 116.0 mm to (187.5, 96.0)
- moved H3 116.0 mm to (149.5, 62.8)
- moved S3 116.0 mm to (149.5, 62.8)
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Connections:
- D1 pad 1: /A2 -> Net-(D1-Pad1)
- D1 pad 2: Net-(D1-Pad2) -> /Col2
- D10 pad 1: /A3 -> Net-(D10-Pad1)
- D10 pad 2: Net-(D10-Pad2) -> /Col1
- D11 pad 1: /A4 -> Net-(D11-Pad1)
- D11 pad 2: Net-(D11-Pad2) -> /Col1
- D12 pad 1: /A4 -> Net-(D12-Pad1)
- D12 pad 2: Net-(D12-Pad2) -> /Col2
- D13 pad 1: /A4 -> Net-(D13-Pad1)
- D13 pad 2: Net-(D13-Pad2) -> /Col3
- D14 pad 1: /A4 -> Net-(D14-Pad1)
- D14 pad 2: Net-(D14-Pad2) -> /Col4
- D15 pad 1: /A4 -> Net-(D15-Pad1)
- D15 pad 2: Net-(D15-Pad2) -> /Col5
- D16 pad 1: /A5 -> Net-(D16-Pad1)
- D16 pad 2: Net-(D16-Pad2) -> /Col5
- D17 pad 1: /A5 -> Net-(D17-Pad1)
- D17 pad 2: Net-(D17-Pad2) -> /Col4
- D18 pad 1: /A5 -> Net-(D18-Pad1)
- D18 pad 2: Net-(D18-Pad2) -> /Col3
- D19 pad 1: /A5 -> Net-(D19-Pad1)
- D19 pad 2: Net-(D19-Pad2) -> /Col2
- D2 pad 1: /A2 -> Net-(D2-Pad1)
- D2 pad 2: Net-(D2-Pad2) -> /Col1
- D20 pad 1: /A5 -> Net-(D20-Pad1)
- D20 pad 2: Net-(D20-Pad2) -> /Col1
- D21 pad 1: /SCK -> Net-(D21-Pad1)
- D21 pad 2: Net-(D21-Pad2) -> /Col1
- D22 pad 1: /SCK -> Net-(D22-Pad1)
- D22 pad 2: Net-(D22-Pad2) -> /Col2
- D23 pad 1: /SCK -> Net-(D23-Pad1)
- D23 pad 2: Net-(D23-Pad2) -> /Col3
- D24 pad 1: /SCK -> Net-(D24-Pad1)
- D24 pad 2: Net-(D24-Pad2) -> /Col4
- D25 pad 1: /SCK -> Net-(D25-Pad1)
- D25 pad 2: Net-(D25-Pad2) -> /Col5
- D3 pad 1: /A2 -> Net-(D3-Pad1)
- D3 pad 2: Net-(D3-Pad2) -> /Col3
- D4 pad 1: /A2 -> Net-(D4-Pad1)
- D4 pad 2: Net-(D4-Pad2) -> /Col4
- D5 pad 1: /A2 -> Net-(D5-Pad1)
- D5 pad 2: Net-(D5-Pad2) -> /Col5
- D6 pad 1: /A3 -> Net-(D6-Pad1)
- D6 pad 2: Net-(D6-Pad2) -> /Col5
- D7 pad 1: /A3 -> Net-(D7-Pad1)
- D7 pad 2: Net-(D7-Pad2) -> /Col4
- D8 pad 1: /A3 -> Net-(D8-Pad1)
- D8 pad 2: Net-(D8-Pad2) -> /Col3
- D9 pad 1: /A3 -> Net-(D9-Pad1)
- D9 pad 2: Net-(D9-Pad2) -> /Col2
- H1 pad 1: Net-(D2-Pad2) -> Net-(D2-Pad1)
- H1 pad 2: /GPIO#3 -> /Row1
- H10 pad 1: Net-(D10-Pad2) -> Net-(D10-Pad1)
- H10 pad 2: /SCL -> /Row2
- H11 pad 1: Net-(D11-Pad2) -> Net-(D11-Pad1)
- H11 pad 2: /GPIO#3 -> /Row3
- H12 pad 1: Net-(D12-Pad2) -> Net-(D12-Pad1)
- H12 pad 2: /GPIO#4 -> /Row3
- H13 pad 1: Net-(D13-Pad2) -> Net-(D13-Pad1)
- H13 pad 2: /GPIO#1 -> /Row3
- H14 pad 1: Net-(D14-Pad2) -> Net-(D14-Pad1)
- H14 pad 2: /SDA -> /Row3
- H15 pad 1: Net-(D15-Pad2) -> Net-(D15-Pad1)
- H15 pad 2: /SCL -> /Row3
- H16 pad 1: Net-(D16-Pad2) -> Net-(D16-Pad1)
- H16 pad 2: /GPIO#3 -> /Row4
- H17 pad 1: Net-(D17-Pad2) -> Net-(D17-Pad1)
- H17 pad 2: /GPIO#4 -> /Row4
- H18 pad 1: Net-(D18-Pad2) -> Net-(D18-Pad1)
- H18 pad 2: /GPIO#1 -> /Row4
- H19 pad 1: Net-(D19-Pad2) -> Net-(D19-Pad1)
- H19 pad 2: /SDA -> /Row4
- H2 pad 1: Net-(D1-Pad2) -> Net-(D1-Pad1)
- H2 pad 2: /GPIO#4 -> /Row1
- H20 pad 1: Net-(D20-Pad2) -> Net-(D20-Pad1)
- H20 pad 2: /SCL -> /Row4
- H21 pad 1: Net-(D21-Pad2) -> Net-(D21-Pad1)
- H21 pad 2: /GPIO#3 -> /Row5
- H22 pad 1: Net-(D22-Pad2) -> Net-(D22-Pad1)
- H22 pad 2: /GPIO#4 -> /Row5
- H23 pad 1: Net-(D23-Pad2) -> Net-(D23-Pad1)
- H23 pad 2: /GPIO#1 -> /Row5
- H24 pad 1: Net-(D24-Pad2) -> Net-(D24-Pad1)
- H24 pad 2: /SDA -> /Row5
- H25 pad 1: Net-(D25-Pad2) -> Net-(D25-Pad1)
- H25 pad 2: /SCL -> /Row5
- H3 pad 1: Net-(D3-Pad2) -> Net-(D3-Pad1)
- H3 pad 2: /GPIO#1 -> /Row1
- H4 pad 1: Net-(D4-Pad2) -> Net-(D4-Pad1)
- H4 pad 2: /SDA -> /Row1
- H5 pad 1: Net-(D5-Pad2) -> Net-(D5-Pad1)
- H5 pad 2: /SCL -> /Row1
- H6 pad 1: Net-(D6-Pad2) -> Net-(D6-Pad1)
- H6 pad 2: /GPIO#3 -> /Row2
- H7 pad 1: Net-(D7-Pad2) -> Net-(D7-Pad1)
- H7 pad 2: /GPIO#4 -> /Row2
- H8 pad 1: Net-(D8-Pad2) -> Net-(D8-Pad1)
- H8 pad 2: /GPIO#1 -> /Row2
- H9 pad 1: Net-(D9-Pad2) -> Net-(D9-Pad1)
- H9 pad 2: /SDA -> /Row2
- S1 pad 1: Net-(D2-Pad2) -> Net-(D2-Pad1)
- S1 pad 2: /GPIO#3 -> /Row1
- S10 pad 1: Net-(D10-Pad2) -> Net-(D10-Pad1)
- S10 pad 2: /SCL -> /Row2
- S11 pad 1: Net-(D11-Pad2) -> Net-(D11-Pad1)
- S11 pad 2: /GPIO#3 -> /Row3
- S12 pad 1: Net-(D12-Pad2) -> Net-(D12-Pad1)
- S12 pad 2: /GPIO#4 -> /Row3
- S13 pad 1: Net-(D13-Pad2) -> Net-(D13-Pad1)
- S13 pad 2: /GPIO#1 -> /Row3
- S14 pad 1: Net-(D14-Pad2) -> Net-(D14-Pad1)
- S14 pad 2: /SDA -> /Row3
- S15 pad 1: Net-(D15-Pad2) -> Net-(D15-Pad1)
- S15 pad 2: /SCL -> /Row3
- S16 pad 1: Net-(D16-Pad2) -> Net-(D16-Pad1)
- S16 pad 2: /GPIO#3 -> /Row4
- S17 pad 1: Net-(D17-Pad2) -> Net-(D17-Pad1)
- S17 pad 2: /GPIO#4 -> /Row4
- S18 pad 1: Net-(D18-Pad2) -> Net-(D18-Pad1)
- S18 pad 2: /GPIO#1 -> /Row4
- S19 pad 1: Net-(D19-Pad2) -> Net-(D19-Pad1)
- S19 pad 2: /SDA -> /Row4
- S2 pad 1: Net-(D1-Pad2) -> Net-(D1-Pad1)
- S2 pad 2: /GPIO#4 -> /Row1
- S20 pad 1: Net-(D20-Pad2) -> Net-(D20-Pad1)
- S20 pad 2: /SCL -> /Row4
- S21 pad 1: Net-(D21-Pad2) -> Net-(D21-Pad1)
- S21 pad 2: /GPIO#3 -> /Row5
- S22 pad 1: Net-(D22-Pad2) -> Net-(D22-Pad1)
- S22 pad 2: /GPIO#4 -> /Row5
- S23 pad 1: Net-(D23-Pad2) -> Net-(D23-Pad1)
- S23 pad 2: /GPIO#1 -> /Row5
- S24 pad 1: Net-(D24-Pad2) -> Net-(D24-Pad1)
- S24 pad 2: /SDA -> /Row5
- S25 pad 1: Net-(D25-Pad2) -> Net-(D25-Pad1)
- S25 pad 2: /SCL -> /Row5
- S3 pad 1: Net-(D3-Pad2) -> Net-(D3-Pad1)
- S3 pad 2: /GPIO#1 -> /Row1
- S4 pad 1: Net-(D4-Pad2) -> Net-(D4-Pad1)
- S4 pad 2: /SDA -> /Row1
- S5 pad 1: Net-(D5-Pad2) -> Net-(D5-Pad1)
- S5 pad 2: /SCL -> /Row1
- S6 pad 1: Net-(D6-Pad2) -> Net-(D6-Pad1)
- S6 pad 2: /GPIO#3 -> /Row2
- S7 pad 1: Net-(D7-Pad2) -> Net-(D7-Pad1)
- S7 pad 2: /GPIO#4 -> /Row2
- S8 pad 1: Net-(D8-Pad2) -> Net-(D8-Pad1)
- S8 pad 2: /GPIO#1 -> /Row2
- S9 pad 1: Net-(D9-Pad2) -> Net-(D9-Pad1)
- S9 pad 2: /SDA -> /Row2
Routing:
- net /SCL: track 280.6 -> 0.00 mm
- net /SDA: track 262.8 -> 0.00 mm
- net /GPIO#1: track 246.9 -> 0.00 mm
- net /USB_1: track 245.3 -> 0.00 mm
- net /Row5: track 0.00 -> 237.8 mm
- net /GPIO#4: track 234.6 -> 0.00 mm
- net /GPIO#2: track 222.8 -> 0.00 mm
- net /Row4: track 0.00 -> 220.0 mm
- net /MI: track 207.0 -> 0.00 mm
- net /Row3: track 0.00 -> 203.1 mm
- net /MO: track 189.1 -> 0.00 mm
- net /Row2: track 0.00 -> 186.0 mm
- net /GPIO#3: track 181.8 -> 0.00 mm
- net /SCK: track 170.6 -> 0.00 mm
- net /A4: track 161.6 -> 0.00 mm
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- added copper zone on F.Cu, net VDD
- added copper zone on B.Cu, net VSS
- removed copper zone on B.Cu, net /GND_1
- removed copper zone on F.Cu, net /USB_1
Other:
- board size 154.3 x 119.4 mm -> 95.2 x 100 mm
- board text added: "WoodElf 01 Hannah Grace '19"
- board text removed: "Wood Elf Prototype 01 Grace 2019"
