File: KiCAD/WoodElf_01/WoodElf_01.sch (KiCad schematic (older format))
At the start: 90 parts, among them J1 AnalogJoystick, M1 MCP23017, M2 MCP23017, M3 MCP23017, P1 ItsyBitsyM4Express, P2 ItsyBitsyM4Express

Commit message: i cant even remember how much i changed here - a lot
Parts:
- removed C26, C27, C28, C29, C30, C31, C32, C33, C34, C35, C36, C37, C38, C39, C40, C41, C42: WS2811, WoodElfLib:WS2811, symbol WoodElf_01-rescue:WS2811
- removed M1, M2, M3: MCP23017, Housings_DIP:DIP-28_W7.62mm, symbol WoodElf_01-rescue:MCP23017
- removed P2: ItsyBitsyM4Express, WoodElfLib:ItsyBitsyM4Express, symbol WoodElf_01-rescue:ItsyBitsyM4Express
- removed R1, R2, R3, R4: 10k, Resistors_SMD:R_2010_HandSoldering, symbol Device:R
- removed S26, S27, S28, S29, S30, S31, S32, S33, S34, S35, S36, S37, S38, S39, S40: Kailh_RGB_Switch, WoodElfLib:SW_Cherry_MX1A_1.00u_PCB, symbol WoodElf_01-rescue:Kailh_RGB_Switch
- added C1, C2: WS2811, WoodElfLib:WS2811, symbol WoodElf_01-rescue:WS2811
- added D1, D10, D11, D12, D13, D14, D15, D16, D17, D18, D19, D2, D20, D21, D22, D23, D24, D25, D3, D4, D5, D6, D7, D8, D9: D, Diode_SMD:D_2010_5025Metric_Pad1.52x2.65mm_HandSolder, symbol Device:D
- added H1, H2: Kailh_HotSwap_SwitchMount, WoodElfLib:Kailh_HotSwap_Socket, symbol WoodElf_01:Kailh_HotSwap_SwitchMount
Connections:
- net Din_2 is gone; now on an unnamed net: C19.6 (DIN)
- net USB_2 is gone; now on net USB_1: C19.8 (VDD), C20.8 (VDD), C21.8 (VDD), C22.8 (VDD), C23.8 (VDD), C24.8 (VDD), C25.8 (VDD), S17.4 (Anode), S18.4 (Anode), S19.4 (Anode), S20.4 (Anode), S21.4 (Anode), S22.4 (Anode), S23.4 (Anode), S24.4 (Anode), S25.4 (Anode)
- net A2: now also D1.1 (K), D2.1 (K), D3.1 (K), D4.1 (K), D5.1 (K); no longer J1.2 (Y)
- net A3: now also D10.1 (K), D6.1 (K), D7.1 (K), D8.1 (K), D9.1 (K); no longer J1.3 (X)
- net Din_1: now also C1.6 (DIN); no longer C3.6 (DIN)
- net GND_1: now also C19.4 (GND), C20.4 (GND), C21.4 (GND), C22.4 (GND), C23.4 (GND), C24.4 (GND), C25.4 (GND), C1.4 (GND), C2.4 (GND); no longer S1.2 (SW_out), S10.2 (SW_out), S11.2 (SW_out), S12.2 (SW_out), S13.2 (SW_out), S14.2 (SW_out), S15.2 (SW_out), S16.2 (SW_out), S2.2 (SW_out), S3.2 (SW_out), S4.2 (SW_out), S5.2 (SW_out), S6.2 (SW_out), S7.2 (SW_out), S8.2 (SW_out), S9.2 (SW_out)
- net USB_1: now also C1.8 (VDD), C2.8 (VDD)
- net at S1.1 (SW_in): now also D1.2 (A)
- net at S2.1 (SW_in): now also D2.2 (A)
- net at S9.1 (SW_in): now also D9.2 (A), H2.1 (Out)
- net at S10.1 (SW_in): now also D10.2 (A)
- net at S11.1 (SW_in): now also D11.2 (A)
- net at S12.1 (SW_in): now also D12.2 (A)
- net at S13.1 (SW_in): now also D13.2 (A)
- net at S14.1 (SW_in): now also D14.2 (A)
- net at S15.1 (SW_in): now also D15.2 (A)
- net at S16.1 (SW_in): now also D16.2 (A)
- net at S3.1 (SW_in): now also D3.2 (A)
- net at S4.1 (SW_in): now also D4.2 (A), H1.1 (Out)
- net at S5.1 (SW_in): now also D5.2 (A)
- net at S6.1 (SW_in): now also D6.2 (A)
- net at S7.1 (SW_in): now also D7.2 (A)
- net at S8.1 (SW_in): now also D8.2 (A)
- net A5: now reaches P1.10 (A5)
- net A5: now also D16.1 (K), D17.1 (K), D18.1 (K), D19.1 (K), D20.1 (K)
- net SCK: now reaches P1.11 (SCK)
- net SCK: now also D21.1 (K), D22.1 (K), D23.1 (K), D24.1 (K), D25.1 (K)
- net GPIO#3: now reaches P1.18 (GPIO#3)
- net GPIO#3: now also S11.2 (SW_out), S16.2 (SW_out), S2.2 (SW_out), S21.2 (SW_out), S6.2 (SW_out)
- net GPIO#4: now reaches P1.19 (GPIO#4)
- net GPIO#4: now also S1.2 (SW_out), S12.2 (SW_out), S17.2 (SW_out), S22.2 (SW_out), S7.2 (SW_out)
- net GPIO#1: now reaches P1.21 (GPIO#1)
- net GPIO#1: now also S13.2 (SW_out), S18.2 (SW_out), S23.2 (SW_out), S3.2 (SW_out), S8.2 (SW_out)
- net A0: now reaches P1.5 (A0)
- net A0: now also J1.2 (Y)
- net A1: now reaches P1.6 (A1)
- net A1: now also J1.3 (X)
- net A4: now reaches P1.9 (A4)
- net A4: now also D11.1 (K), D12.1 (K), D13.1 (K), D14.1 (K), D15.1 (K)
- net at S2.3 (LED_R): now also C1.1 (outR); no longer C4.1 (outR)
- net at S2.5 (LED_G): now also C1.2 (outG); no longer C4.2 (outG)
- net at S2.6 (LED_B): now also C1.3 (outB); no longer C4.3 (outB)
- net at S3.3 (LED_R): now also C2.1 (outR); no longer C5.1 (outR)
- net at S3.5 (LED_G): now also C2.2 (outG); no longer C5.2 (outG)
- net at S3.6 (LED_B): now also C2.3 (outB); no longer C5.3 (outB)
- net at S4.3 (LED_R): now also C4.1 (outR); no longer C6.1 (outR)
- net at S4.5 (LED_G): now also C4.2 (outG); no longer C6.2 (outG)
- net at S4.6 (LED_B): now also C4.3 (outB); no longer C6.3 (outB)
- net at S5.3 (LED_R): now also C5.1 (outR); no longer C7.1 (outR)
- net at S5.5 (LED_G): now also C5.2 (outG); no longer C7.2 (outG)
- net at S5.6 (LED_B): now also C5.3 (outB); no longer C7.3 (outB)
- net at S6.3 (LED_R): now also C6.1 (outR); no longer C8.1 (outR)
- net at S6.5 (LED_G): now also C6.2 (outG); no longer C8.2 (outG)
- net at S6.6 (LED_B): now also C6.3 (outB); no longer C8.3 (outB)
- net at S7.3 (LED_R): now also C7.1 (outR); no longer C9.1 (outR)
- net at S7.5 (LED_G): now also C7.2 (outG); no longer C9.2 (outG)
- net at S7.6 (LED_B): now also C7.3 (outB); no longer C9.3 (outB)
- net at S8.3 (LED_R): now also C8.1 (outR); no longer C10.1 (outR)
- net at S8.5 (LED_G): now also C8.2 (outG); no longer C10.2 (outG)
- net at S8.6 (LED_B): now also C8.3 (outB); no longer C10.3 (outB)
- net at S9.3 (LED_R): now also C9.1 (outR); no longer C11.1 (outR)
- net at S9.5 (LED_G): now also C9.2 (outG); no longer C11.2 (outG)
- net at S9.6 (LED_B): now also C9.3 (outB); no longer C11.3 (outB)
- net at S10.3 (LED_R): now also C10.1 (outR); no longer C12.1 (outR)
- net at S10.5 (LED_G): now also C10.2 (outG); no longer C12.2 (outG)
- net at S10.6 (LED_B): now also C10.3 (outB); no longer C12.3 (outB)
- net at S11.3 (LED_R): now also C11.1 (outR); no longer C13.1 (outR)
- net at S11.5 (LED_G): now also C11.2 (outG); no longer C13.2 (outG)
- net at S11.6 (LED_B): now also C11.3 (outB); no longer C13.3 (outB)
- net at S12.3 (LED_R): now also C12.1 (outR); no longer C14.1 (outR)
- net at S12.5 (LED_G): now also C12.2 (outG); no longer C14.2 (outG)
- net at S12.6 (LED_B): now also C12.3 (outB); no longer C14.3 (outB)
- net at S13.3 (LED_R): now also C13.1 (outR); no longer C15.1 (outR)
- net at S13.5 (LED_G): now also C13.2 (outG); no longer C15.2 (outG)
- net at S13.6 (LED_B): now also C13.3 (outB); no longer C15.3 (outB)
- net at S14.3 (LED_R): now also C14.1 (outR); no longer C16.1 (outR)
- net at S14.5 (LED_G): now also C14.2 (outG); no longer C16.2 (outG)
- net at S14.6 (LED_B): now also C14.3 (outB); no longer C16.3 (outB)
- net at S15.3 (LED_R): now also C15.1 (outR); no longer C17.1 (outR)
- net at S15.5 (LED_G): now also C15.2 (outG); no longer C17.2 (outG)
- net at S15.6 (LED_B): now also C15.3 (outB); no longer C17.3 (outB)
- net at S16.3 (LED_R): now also C16.1 (outR); no longer C18.1 (outR)
- net at S16.5 (LED_G): now also C16.2 (outG); no longer C18.2 (outG)
- net at S16.6 (LED_B): now also C16.3 (outB); no longer C18.3 (outB)
- net at S17.1 (SW_in): now also D17.2 (A)
- net at S17.3 (LED_R): now also C17.1 (outR); no longer C19.1 (outR)
- net at S17.5 (LED_G): now also C17.2 (outG); no longer C19.2 (outG)
- net at S17.6 (LED_B): now also C17.3 (outB); no longer C19.3 (outB)
- net at S18.1 (SW_in): now also D18.2 (A)
- net at S18.3 (LED_R): now also C18.1 (outR); no longer C20.1 (outR)
- net at S18.5 (LED_G): now also C18.2 (outG); no longer C20.2 (outG)
- net at S18.6 (LED_B): now also C18.3 (outB); no longer C20.3 (outB)
- net at S19.1 (SW_in): now also D19.2 (A)
- net at S19.3 (LED_R): now also C19.1 (outR); no longer C21.1 (outR)
- net at S19.5 (LED_G): now also C19.2 (outG); no longer C21.2 (outG)
- net at S19.6 (LED_B): now also C19.3 (outB); no longer C21.3 (outB)
- net at S20.1 (SW_in): now also D20.2 (A)
- net at S20.3 (LED_R): now also C20.1 (outR); no longer C22.1 (outR)
- net at S20.5 (LED_G): now also C20.2 (outG); no longer C22.2 (outG)
- net at S20.6 (LED_B): now also C20.3 (outB); no longer C22.3 (outB)
- net at S21.1 (SW_in): now also D21.2 (A)
- net at S21.3 (LED_R): now also C21.1 (outR); no longer C23.1 (outR)
- net at S21.5 (LED_G): now also C21.2 (outG); no longer C23.2 (outG)
- net at S21.6 (LED_B): now also C21.3 (outB); no longer C23.3 (outB)
- net at S25.1 (SW_in): now also D25.2 (A)
- net at S22.1 (SW_in): now also D22.2 (A)
- net at S23.1 (SW_in): now also D23.2 (A)
- net at S24.1 (SW_in): now also D24.2 (A)
- net at S22.3 (LED_R): now also C22.1 (outR); no longer C24.1 (outR)
- net at S22.5 (LED_G): now also C22.2 (outG); no longer C24.2 (outG)
- net at S22.6 (LED_B): now also C22.3 (outB); no longer C24.3 (outB)
- net at S23.3 (LED_R): now also C23.1 (outR); no longer C25.1 (outR)
- net at S23.5 (LED_G): now also C23.2 (outG); no longer C25.2 (outG)
- net at S23.6 (LED_B): now also C23.3 (outB); no longer C25.3 (outB)
- net at S24.3 (LED_R): now also C24.1 (outR)
- net at S24.5 (LED_G): now also C24.2 (outG)
- net at S24.6 (LED_B): now also C24.3 (outB)
- net at S25.3 (LED_R): now also C25.1 (outR)
- net at S25.5 (LED_G): now also C25.2 (outG)
- net at S25.6 (LED_B): now also C25.3 (outB)
- net at C3.5 (DO): now also C2.6 (DIN); no longer C4.6 (DIN)
- removed net GND_2: C19.4 (GND), C20.4 (GND), C21.4 (GND), C22.4 (GND), C23.4 (GND), C24.4 (GND), C25.4 (GND), S17.2 (SW_out), S18.2 (SW_out), S19.2 (SW_out), S20.2 (SW_out), S21.2 (SW_out), S22.2 (SW_out), S23.2 (SW_out), S24.2 (SW_out), S25.2 (SW_out)
- net SCL_1 renamed SCL
- net SCL: now also S10.2 (SW_out), S15.2 (SW_out), S20.2 (SW_out), S25.2 (SW_out), S5.2 (SW_out)
- net SDA_1 renamed SDA
- net SDA: now also S14.2 (SW_out), S19.2 (SW_out), S24.2 (SW_out), S4.2 (SW_out), S9.2 (SW_out), H1.2 (In), H2.2 (In)
- new net: C1.5 (DO), C3.6 (DIN)
- new net: C2.5 (DO), C4.6 (DIN)
- no-connect marks 94 -> 33
Other:
- moved on the sheet: C3, J1, P1, S1

Commit message: fleshing out some more of the pcb
Parts:
- added C26, C27, C28, C29, C30, C31, C32, C33, C34, C35, C36, C37, C38, C39, C40: WS2811, WoodElfLib:WS2811, symbol WoodElf_01-rescue:WS2811
- added D26, D27, D28, D29, D30, D31, D32, D33, D34, D35, D36, D37, D38, D39, D40: D, Diode_SMD:D_2010_5025Metric_Pad1.52x2.65mm_HandSolder, symbol Device:D
- added H1, H10, H11, H12, H13, H14, H15, H16, H17, H18, H19, H20, H21, H22, H23, H24, H25, H26, H27, H28, H29, H3, H30, H31, H32, H33, H34, H35, H36, H37, H38, H39, H40, H5, H6, H7, H8, H9: Kailh_HotSwap_SwitchMount, WoodElfLib:Kailh_HotSwap_Socket, symbol WoodElf_01:Kailh_HotSwap_SwitchMount
- added S26, S27, S28, S29, S30, S31, S32, S33, S34, S35, S36, S37, S38, S39, S40: Kailh_RGB_Switch, WoodElfLib:SW_Cherry_MX1A_1.00u_PCB, symbol WoodElf_01-rescue:Kailh_RGB_Switch
- renumbered H1 to H4, S2 to S1, S1 to S2
Connections:
- net GND_1: now also C26.4 (GND), C27.4 (GND), C28.4 (GND), C29.4 (GND), C30.4 (GND), C31.4 (GND), C32.4 (GND), C33.4 (GND), C34.4 (GND), C35.4 (GND), C36.4 (GND), C37.4 (GND), C38.4 (GND), C39.4 (GND), C40.4 (GND)
- net GPIO#1: now also H13.2 (In), H18.2 (In), H23.2 (In), H28.2 (In), H3.2 (In), H33.2 (In), H38.2 (In), H8.2 (In), S28.2 (SW_out), S33.2 (SW_out), S38.2 (SW_out)
- net GPIO#3: now also H1.2 (In), H11.2 (In), H16.2 (In), H21.2 (In), H26.2 (In), H31.2 (In), H36.2 (In), H6.2 (In), S26.2 (SW_out), S31.2 (SW_out), S36.2 (SW_out)
- net GPIO#4: now also H2.2 (In), H12.2 (In), H17.2 (In), H22.2 (In), H27.2 (In), H32.2 (In), H37.2 (In), H7.2 (In), S27.2 (SW_out), S32.2 (SW_out), S37.2 (SW_out)
- net SCL: now also H10.2 (In), H15.2 (In), H20.2 (In), H25.2 (In), H30.2 (In), H35.2 (In), H40.2 (In), H5.2 (In), S30.2 (SW_out), S35.2 (SW_out), S40.2 (SW_out)
- net SDA: now also H14.2 (In), H19.2 (In), H24.2 (In), H29.2 (In), H34.2 (In), H39.2 (In), H9.2 (In), S29.2 (SW_out), S34.2 (SW_out), S39.2 (SW_out); no longer H2.2 (In)
- net USB_1: now also C26.8 (VDD), C27.8 (VDD), C28.8 (VDD), C29.8 (VDD), C30.8 (VDD), C31.8 (VDD), C32.8 (VDD), C33.8 (VDD), C34.8 (VDD), C35.8 (VDD), C36.8 (VDD), C37.8 (VDD), C38.8 (VDD), C39.8 (VDD), C40.8 (VDD), S26.4 (Anode), S27.4 (Anode), S28.4 (Anode), S29.4 (Anode), S30.4 (Anode), S31.4 (Anode), S32.4 (Anode), S33.4 (Anode), S34.4 (Anode), S35.4 (Anode), S36.4 (Anode), S37.4 (Anode), S38.4 (Anode), S39.4 (Anode), S40.4 (Anode)
- net MO: now reaches P1.12 (MO)
- net MO: now also D26.1 (K), D27.1 (K), D28.1 (K), D29.1 (K), D30.1 (K)
- net MI: now reaches P1.13 (MI)
- net MI: now also D31.1 (K), D32.1 (K), D33.1 (K), D34.1 (K), D35.1 (K)
- net GPIO#2: now reaches P1.14 (GPIO#2)
- net GPIO#2: now also D36.1 (K), D37.1 (K), D38.1 (K), D39.1 (K), D40.1 (K)
- net at D1.2 (A), S2.1 (SW_in): now also H2.1 (Out)
- net at D2.2 (A), S1.1 (SW_in): now also H1.1 (Out)
- net at D3.2 (A), S3.1 (SW_in): now also H3.1 (Out)
- net at D5.2 (A), S5.1 (SW_in): now also H5.1 (Out)
- net at D7.2 (A), S7.1 (SW_in): now also H7.1 (Out)
- net at D6.2 (A), S6.1 (SW_in): now also H6.1 (Out)
- net at D9.2 (A), S9.1 (SW_in): now also H9.1 (Out); no longer H2.1 (Out)
- net at D8.2 (A), S8.1 (SW_in): now also H8.1 (Out)
- net at D10.2 (A), S10.1 (SW_in): now also H10.1 (Out)
- net at D12.2 (A), S12.1 (SW_in): now also H12.1 (Out)
- net at D11.2 (A), S11.1 (SW_in): now also H11.1 (Out)
- net at D14.2 (A), S14.1 (SW_in): now also H14.1 (Out)
- net at D13.2 (A), S13.1 (SW_in): now also H13.1 (Out)
- net at D15.2 (A), S15.1 (SW_in): now also H15.1 (Out)
- net at D17.2 (A), S17.1 (SW_in): now also H17.1 (Out)
- net at D16.2 (A), S16.1 (SW_in): now also H16.1 (Out)
- net at D19.2 (A), S19.1 (SW_in): now also H19.1 (Out)
- net at D18.2 (A), S18.1 (SW_in): now also H18.1 (Out)
- net at D20.2 (A), S20.1 (SW_in): now also H20.1 (Out)
- net at D22.2 (A), S22.1 (SW_in): now also H22.1 (Out)
- net at D21.2 (A), S21.1 (SW_in): now also H21.1 (Out)
- net at D24.2 (A), S24.1 (SW_in): now also H24.1 (Out)
- net at D23.2 (A), S23.1 (SW_in): now also H23.1 (Out)
- net at D25.2 (A), S25.1 (SW_in): now also H25.1 (Out)
- net at C25.5 (DO): now also C26.6 (DIN)
- new net: D27.2 (A), H27.1 (Out), S27.1 (SW_in)
- new net: C27.1 (outR), S27.3 (LED_R)
- new net: C27.2 (outG), S27.5 (LED_G)
- new net: C27.3 (outB), S27.6 (LED_B)
- new net: C27.5 (DO), C28.6 (DIN)
- new net: C26.5 (DO), C27.6 (DIN)
- new net: D26.2 (A), H26.1 (Out), S26.1 (SW_in)
- new net: C26.1 (outR), S26.3 (LED_R)
- new net: C26.2 (outG), S26.5 (LED_G)
- new net: C26.3 (outB), S26.6 (LED_B)
- new net: D29.2 (A), H29.1 (Out), S29.1 (SW_in)
- new net: C29.1 (outR), S29.3 (LED_R)
- new net: C29.2 (outG), S29.5 (LED_G)
- new net: C29.3 (outB), S29.6 (LED_B)
- new net: C29.5 (DO), C30.6 (DIN)
- new net: C28.5 (DO), C29.6 (DIN)
- new net: D28.2 (A), H28.1 (Out), S28.1 (SW_in)
- new net: C28.1 (outR), S28.3 (LED_R)
- new net: C28.2 (outG), S28.5 (LED_G)
- new net: C28.3 (outB), S28.6 (LED_B)
- new net: D30.2 (A), H30.1 (Out), S30.1 (SW_in)
- new net: C30.1 (outR), S30.3 (LED_R)
- new net: C30.2 (outG), S30.5 (LED_G)
- new net: C30.3 (outB), S30.6 (LED_B)
- new net: C30.5 (DO), C31.6 (DIN)
- new net: D32.2 (A), H32.1 (Out), S32.1 (SW_in)
- new net: C32.1 (outR), S32.3 (LED_R)
- new net: C32.2 (outG), S32.5 (LED_G)
- new net: C32.3 (outB), S32.6 (LED_B)
- new net: C32.5 (DO), C33.6 (DIN)
- new net: C31.5 (DO), C32.6 (DIN)
- new net: D31.2 (A), H31.1 (Out), S31.1 (SW_in)
- new net: C31.1 (outR), S31.3 (LED_R)
- new net: C31.2 (outG), S31.5 (LED_G)
- new net: C31.3 (outB), S31.6 (LED_B)
- new net: D34.2 (A), H34.1 (Out), S34.1 (SW_in)
- new net: C34.1 (outR), S34.3 (LED_R)
- new net: C34.2 (outG), S34.5 (LED_G)
- new net: C34.3 (outB), S34.6 (LED_B)
- new net: C34.5 (DO), C35.6 (DIN)
- new net: C33.5 (DO), C34.6 (DIN)
- new net: D33.2 (A), H33.1 (Out), S33.1 (SW_in)
- new net: C33.1 (outR), S33.3 (LED_R)
- new net: C33.2 (outG), S33.5 (LED_G)
- new net: C33.3 (outB), S33.6 (LED_B)
- new net: D35.2 (A), H35.1 (Out), S35.1 (SW_in)
- new net: C35.1 (outR), S35.3 (LED_R)
- new net: C35.2 (outG), S35.5 (LED_G)
- new net: C35.3 (outB), S35.6 (LED_B)
- new net: C35.5 (DO), C36.6 (DIN)
- new net: D37.2 (A), H37.1 (Out), S37.1 (SW_in)
- new net: C37.1 (outR), S37.3 (LED_R)
- new net: C37.2 (outG), S37.5 (LED_G)
- new net: C37.3 (outB), S37.6 (LED_B)
- new net: C37.5 (DO), C38.6 (DIN)
- new net: C36.5 (DO), C37.6 (DIN)
- new net: D36.2 (A), H36.1 (Out), S36.1 (SW_in)
- new net: C36.1 (outR), S36.3 (LED_R)
- new net: C36.2 (outG), S36.5 (LED_G)
- new net: C36.3 (outB), S36.6 (LED_B)
- new net: D39.2 (A), H39.1 (Out), S39.1 (SW_in)
- new net: C39.1 (outR), S39.3 (LED_R)
- new net: C39.2 (outG), S39.5 (LED_G)
- new net: C39.3 (outB), S39.6 (LED_B)
- new net: C39.5 (DO), C40.6 (DIN)
- new net: C38.5 (DO), C39.6 (DIN)
- new net: D38.2 (A), H38.1 (Out), S38.1 (SW_in)
- new net: C38.1 (outR), S38.3 (LED_R)
- new net: C38.2 (outG), S38.5 (LED_G)
- new net: C38.3 (outB), S38.6 (LED_B)
- new net: D40.2 (A), H40.1 (Out), S40.1 (SW_in)
- new net: C40.1 (outR), S40.3 (LED_R)
- new net: C40.2 (outG), S40.5 (LED_G)
- new net: C40.3 (outB), S40.6 (LED_B)
- no-connect marks 33 -> 55
Other:
- moved on the sheet: D1, D2, D3, D5

Commit message: Started on a full-size PCB
Parts:
- removed C1, C10, C11, C12, C13, C14, C15, C16, C17, C18, C19, C2, C20, C21, C22, C23, C24, C25, C26, C27, C28, C29, C3, C30, C31, C32, C33, C34, C35, C36, C37, C38, C39, C4, C40, C5, C6, C7, C8, C9: WS2811, WoodElfLib:WS2811, symbol WoodElf_01-rescue:WS2811
- removed D1, D10, D11, D12, D13, D14, D15, D16, D17, D18, D19, D2, D20, D21, D22, D23, D24, D25, D26, D27, D28, D29, D3, D30, D31, D32, D33, D34, D35, D36, D37, D38, D39, D4, D40, D5, D6, D7, D8, D9: D, Diode_SMD:D_2010_5025Metric_Pad1.52x2.65mm_HandSolder, symbol Device:D
- removed H1, H10, H11, H12, H13, H14, H15, H16, H17, H18, H19, H2, H20, H21, H22, H23, H24, H25, H26, H27, H28, H29, H3, H30, H31, H32, H33, H34, H35, H36, H37, H38, H39, H4, H40, H5, H6, H7, H8, H9: Kailh_HotSwap_SwitchMount, WoodElfLib:Kailh_HotSwap_Socket, symbol WoodElf_01:Kailh_HotSwap_SwitchMount
- removed J1: AnalogJoystick, WoodElfLib:Joystick, symbol WoodElf_01-rescue:AnalogJoystick-RESCUE-WoodElf_01
- removed P1: ItsyBitsyM4Express, WoodElfLib:ItsyBitsyM4Express, symbol WoodElf_01-rescue:ItsyBitsyM4Express
- removed S1, S10, S11, S12, S13, S14, S15, S16, S17, S18, S19, S2, S20, S21, S22, S23, S24, S25, S26, S27, S28, S29, S3, S30, S31, S32, S33, S34, S35, S36, S37, S38, S39, S4, S40, S5, S6, S7, S8, S9: Kailh_RGB_Switch, WoodElfLib:SW_Cherry_MX1A_1.00u_PCB, symbol WoodElf_01-rescue:Kailh_RGB_Switch
- added T1, T10, T11, T12, T13, T2, T3, T4, T5, T6, T7, T8, T9: BlankThrough-Hole, WoodElf_Lib:BlankThrough-Hole, symbol WoodElf_01:BlankThrough-Hole
Connections:
- new net Col1: T1.1 (In)
- new net Col2: T2.1 (In)
- new net Col3: T3.1 (In)
- new net Col4: T4.1 (In)
- new net Col5: T5.1 (In)
- new net Din: T11.1 (In)
- new net Row1: T6.1 (In)
- new net Row2: T7.1 (In)
- new net Row3: T8.1 (In)
- new net Row4: T9.1 (In)
- new net Row5: T10.1 (In)
- new net VDD: T12.1 (In)
- new net VSS: T13.1 (In)
- no-connect marks 55 -> 1

Commit message: completely redid everything
properly this time.
Parts:
- removed T10: BlankThrough-Hole, WoodElf_Lib:BlankThrough-Hole, symbol WoodElf_01:BlankThrough-Hole
- added T6: BlankThrough-Hole, WoodElf_Lib:BlankThrough-Hole, symbol WoodElf_01:BlankThrough-Hole
- renumbered T9 to T10, T11 to T12, T12 to T13, T13 to T14, T6 to T7, T7 to T8, T8 to T9
Connections:
- new net Col6: T6.1 (In)
Other:
- moved on the sheet: T1, T2, T3, T4, T5
